File: Hardware/MainPCB/MainPCB.kicad_pcb (KiCad board)
At the start: 2 copper layers, 99.1 x 103.9 mm, 53 parts, among them J1 USB_B_Micro, J2 Conn_01x09_Female, J3 UART, Q1 NTR2101P, Q2 FDS9926A, U1 BQ24075, U2 BQ29700, U3 TLV75533PDBV, U4 ESP32-WROOM-32D, U5 TPS22919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

Commit message: probleemke?
Parts:
- J2: value Conn_01x09_Female -> Conn_01x11_Male; footprint Connector_PinHeader_2.54mm:PinHeader_1x09_P2.54mm_Vertical -> Connector_PinHeader_1.00mm:PinHeader_1x11_P1.00mm_Vertical
- moved C12 62.6 mm to (118.1, 116.8)
- moved J3 59.7 mm to (146.1, 133.3), turned to 270 degrees
- moved R13 54.8 mm to (100.3, 102.9), turned to 270 degrees
- moved C16 50.2 mm to (95.2, 97.8), turned to 270 degrees
- moved R12 47.7 mm to (114.3, 99.1), turned to 270 degrees
- moved R14 43.3 mm to (91.4, 102.9), turned to 270 degrees
- moved C15 42.9 mm to (113.0, 105.4)
- moved C18 42.8 mm to (101.6, 109.2), turned to 180 degrees
- moved U5 35.2 mm to (110.5, 97.8), turned to 0 degrees
- moved C17 33.2 mm to (85.1, 97.8), turned to 270 degrees
- moved U6 31.6 mm to (100.3, 97.8)
- moved C14 30.2 mm to (105.4, 97.8), turned to 270 degrees
- moved BOOT1 27.8 mm to (118.1, 129.5), turned to 270 degrees
- moved C19 23.6 mm to (89.4, 108.0), turned to 180 degrees
- moved J2 22.9 mm to (112.7, 115.6), turned to 270 degrees
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Connections:
- C15 pad 1: Net-(C15-Pad1) -> PowerOutS1
- C18 pad 1: Net-(C18-Pad1) -> PowerOutS2
- C19 pad 1: Net-(C19-Pad1) -> PowerOutS3
- J2 pad 1: Detector_out -> +3V3
- J2 pad 2: AUX -> SDA
- J2 pad 3: nWake -> SCL
- J2 pad 4: Int_CCSB11 -> Int_AMG8833
- J2 pad 5: Int_AMG8833 -> GND
- J2 pad 6: GND -> Int_CCSB11
- J2 pad 7: SCL -> nWake
- J2 pad 8: SDA -> Detector_out
- J2 pad 9: +3V3 -> PowerOutS1
- R12 pad 1: Net-(C15-Pad1) -> PowerOutS1
- R13 pad 1: Net-(C18-Pad1) -> PowerOutS2
- R14 pad 1: Net-(C19-Pad1) -> PowerOutS3
- U4 pad 23: PowerS1 -> Net-(U4-Pad23)
- U4 pad 29: Net-(U4-Pad29) -> PowerS1
- U4 pad 6: AUX -> Net-(U4-Pad6)
- U5 pad 6: Net-(C15-Pad1) -> PowerOutS1
- U6 pad 6: Net-(C18-Pad1) -> PowerOutS2
- U7 pad 6: Net-(C19-Pad1) -> PowerOutS3
Other:
- board size 99.1 x 103.9 mm -> 99.1 x 100.3 mm
