File: Hardware/MainPCB/MainPCB.sch (KiCad schematic (older format))
At the start: 31 parts, among them J1 USB_B_Micro, Q1 NTR2101P, Q2 FDS9926A, U1 BQ24075, U2 BQ29700, U3 TLV75533PDBV

Commit message: Aux pin verwijderd + aanpassing gedaan VSS naar -VBAT en GND op de juiste plaats gezet
Connections:
- net GND: now also C1.2, C2.2, C4.2, C5.2, J1.5 (GND), J1.6 (Shield), R1.2, R2.2, R3.2, R4.2, R8.2, U1.15 (SYSOFF), U1.17 (PAD), U1.4 (~CE), U1.6 (EN1), U1.8 (VSS)
- removed net VSS: C1.2, C2.2, C3.2, C4.2, C5.2, C6.2, C7.2, C8.2, J1.5 (GND), J1.6 (Shield), JP1.2, Q1.1 (G), Q2.3 (S2), R1.2, R10.2, R2.2, R3.2, R4.2, R8.2, U1.15 (SYSOFF), U1.17 (PAD), U1.4 (~CE), U1.6 (EN1), U1.8 (VSS), U2.4 (VSS)
- new net -BATT: C6.2, C7.2, C8.2, JP1.2, Q1.1 (G), Q2.3 (S2), R10.2, U2.4 (VSS)
Changed lines of the file:
@@
 Wire Wire Line
 	3500 4200 3300 4200
-$Comp
-L power:VSS #PWR012
-U 1 1 5E5F32D4
-P 3500 4950
-F 0 "#PWR012" H 3500 4800 50  0001 C CNN
-F 1 "VSS" H 3518 5123 50  0000 C CNN
-F 2 "" H 3500 4950 50  0001 C CNN
-F 3 "" H 3500 4950 50  0001 C CNN
-	1    3500 4950
-	-1   0    0    1
-$EndComp
-$Comp
-L power:VSS #PWR08
-U 1 1 5E5F44D7
-P 2650 4850
-F 0 "#PWR08" H 2650 4700 50  0001 C CNN
-F 1 "VSS" H 2668 5023 50  0000 C CNN
-F 2 "" H 2650 4850 50  0001 C CNN
-F 3 "" H 2650 4850 50  0001 C CNN
-	1    2650 4850
-	-1   0    0    1
-$EndComp
-$Comp
-L power:VSS #PWR06
-U 1 1 5E5F485B
-P 2000 5000
-F 0 "#PWR06" H 2000 4850 50  0001 C CNN
-F 1 "VSS" H 2018 5173 50  0000 C CNN
-F 2 "" H 2000 5000 50  0001 C CNN
-F 3 "" H 2000 5000 50  0001 C CNN
-	1    2000 5000
-	-1   0    0    1
-$EndComp
-$Comp
-L power:VSS #PWR04
-U 1 1 5E5F4CA8
-P 1600 5000
-F 0 "#PWR04" H 1600 4850 50  0001 C CNN
-F 1 "VSS" H 1618 5173 50  0000 C CNN
-F 2 "" H 1600 5000 50  0001 C CNN
-F 3 "" H 1600 5000 50  0001 C CNN
-	1    1600 5000
-	-1   0    0    1
-$EndComp
 Wire Wire Line
 	3500 4950 3500 4900
-$Comp
-L power:VSS #PWR03
-U 1 1 5E5F6330
-P 1400 4300
-F 0 "#PWR03" H 1400 4150 50  0001 C CNN
-F 1 "VSS" H 1418 4473 50  0000 C CNN
-F 2 "" H 1400 4300 50  0001 C CNN
-F 3 "" H 1400 4300 50  0001 C CNN
-	1    1400 4300
-	-1   0    0    1
-$EndComp
-$Comp
-L power:VSS #PWR010
-U 1 1 5E5F6B13
-P 3450 2100
-F 0 "#PWR010" H 3450 1950 50  0001 C CNN
-F 1 "VSS" H 3468 2273 50  0000 C CNN
-F 2 "" H 3450 2100 50  0001 C CNN
-F 3 "" H 3450 2100 50  0001 C CNN
-	1    3450 2100
-	-1   0    0    1
-$EndComp
 $Comp
 L Device:C C3
@@
 Text GLabel 2300 2900 0    50   Input ~ 0
 Vin
-$Comp
-L power:VSS #PWR021
-U 1 1 5E618086
-P 6450 4000
-F 0 "#PWR021" H 6450 3850 50  0001 C CNN
-F 1 "VSS" H 6468 4173 50  0000 C CNN
-F 2 "" H 6450 4000 50  0001 C CNN
-F 3 "" H 6450 4000 50  0001 C CNN
-	1    6450 4000
-	-1   0    0    1
-$EndComp
 Wire Wire Line
 	2700 2900 2400 2900
 Wire Wire Line
 	2700 2900 2700 3500
-$Comp
-L power:VSS #PWR07
-U 1 1 5E61F3C2
-P 2400 3300
-F 0 "#PWR07" H 2400 3150 50  0001 C CNN
-F 1 "VSS" H 2418 3473 50  0000 C CNN
-F 2 "" H 2400 3300 50  0001 C CNN
-F 3 "" H 2400 3300 50  0001 C CNN
-	1    2400 3300
-	-1   0    0    1
-$EndComp
 Wire Wire Line
 	2400 3300 2400 3250
@@
 Wire Wire Line
 	5500 3400 5500 3450
-$Comp
-L power:VSS #PWR018
-U 1 1 5E627A24
-P 5500 3800
-F 0 "#PWR018" H 5500 3650 50  0001 C CNN
-F 1 "VSS" H 5518 3973 50  0000 C CNN
-F 2 "" H 5500 3800 50  0001 C CNN
-F 3 "" H 5500 3800 50  0001 C CNN
-	1    5500 3800
-	-1   0    0    1
-$EndComp
 Wire Wire Line
 	5500 3800 5500 3750
@@
 	1    0    0    -1
 $EndComp
-$Comp
-L power:VSS #PWR015
-U 1 1 5E630A70
-P 3850 4250
-F 0 "#PWR015" H 3850 4100 50  0001 C CNN
-F 1 "VSS" H 3750 4300 50  0000 C CNN
-F 2 "" H 3850 4250 50  0001 C CNN
-F 3 "" H 3850 4250 50  0001 C CNN
-	1    3850 4250
-	-1   0    0    1
-$EndComp
 Wire Wire Line
 	3300 4500 4650 4500
@@
 	1    0    0    -1
 $EndComp
-$Comp
-L power:VSS #PWR013
-U 1 1 5E6463B0
-P 3600 3750
-F 0 "#PWR013" H 3600 3600 50  0001 C CNN
-F 1 "VSS" H 3650 3900 50  0000 C CNN
-F 2 "" H 3600 3750 50  0001 C CNN
-F 3 "" H 3600 3750 50  0001 C CNN
-	1    3600 3750
-	-1   0    0    1
-$EndComp
 Wire Wire Line
 	3600 3450 3450 3450
@@
 Text GLabel 2500 1000 2    50   Input ~ 0
 Vin
-$Comp
-L power:VSS #PWR05
-U 1 1 5E64C076
-P 2000 1450
-F 0 "#PWR05" H 2000 1300 50  0001 C CNN
-F 1 "VSS" H 2018 1623 50  0000 C CNN
-F 2 "" H 2000 1450 50  0001 C CNN
-F 3 "" H 2000 1450 50  0001 C CNN
-	1    2000 1450
-	-1   0    0    1
-$EndComp
 $Comp
 L Device:C C1
@@
 Wire Wire Line
 	5950 3600 5950 3650
-$Comp
-L power:VSS #PWR020
-U 1 1 5E656439
-P 5950 4000
-F 0 "#PWR020" H 5950 3850 50  0001 C CNN
-F 1 "VSS" H 5968 4173 50  0000 C CNN
-F 2 "" H 5950 4000 50  0001 C CNN
-F 3 "" H 5950 4000 50  0001 C CNN
-	1    5950 4000
-	-1   0    0    1
-$EndComp
-Wire Wire Line
-	5950 4000 5950 3950
 Wire Wire Line
 	6450 3800 6450 4000
-$Comp
-L power:VSS #PWR023
-U 1 1 5E65BF35
-P 8050 4300
-F 0 "#PWR023" H 8050 4150 50  0001 C CNN
-F 1 "VSS" H 8068 4473 50  0000 C CNN
-F 2 "" H 8050 4300 50  0001 C CNN
-F 3 "" H 8050 4300 50  0001 C CNN
-	1    8050 4300
-	-1   0    0    1
-$EndComp
 $Comp
 L power:GND #PWR022
@@
 Wire Wire Line
 	1550 1000 2000 1000
-$Comp
-L power:VSS #PWR01
-U 1 1 5E70438C
-P 1200 1700
-F 0 "#PWR01" H 1200 1550 50  0001 C CNN
-F 1 "VSS" H 1218 1873 50  0000 C CNN
-F 2 "" H 1200 1700 50  0001 C CNN
-F 3 "" H 1200 1700 50  0001 C CNN
-	1    1200 1700
-	-1   0    0    1
-$EndComp
 Wire Wire Line
 	1200 1700 1200 1650
@@
 Wire Wire Line
 	1400 4000 1400 4100
-$Comp
-L power:VSS #PWR042
-U 1 1 5E684144
-P 4950 1400
-F 0 "#PWR042" H 4950 1250 50  0001 C CNN
-F 1 "VSS" H 4968 1573 50  0000 C CNN
-F 2 "" H 4950 1400 50  0001 C CNN
-F 3 "" H 4950 1400 50  0001 C CNN
-	1    4950 1400
-	-1   0    0    1
-$EndComp
 Wire Wire Line
 	4950 1400 4950 1300
@@
 Wire Wire Line
 	3450 1300 3450 1450
+$Comp
+L power:-BATT #PWR0101
+U 1 1 5E6695A7
+P 3450 2100
+F 0 "#PWR0101" H 3450 1950 50  0001 C CNN
+F 1 "-BATT" H 3465 2273 50  0000 C CNN
+F 2 "" H 3450 2100 50  0001 C CNN
+F 3 "" H 3450 2100 50  0001 C CNN
+	1    3450 2100
+	-1   0    0    1
+$EndComp
+$Comp
+L power:-BATT #PWR0102
+U 1 1 5E66A572
+P 4950 1400
+F 0 "#PWR0102" H 4950 1250 50  0001 C CNN
+F 1 "-BATT" H 4965 1573 50  0000 C CNN
+F 2 "" H 4950 1400 50  0001 C CNN
+F 3 "" H 4950 1400 50  0001 C CNN
+	1    4950 1400
+	-1   0    0    1
+$EndComp
+$Comp
+L power:-BATT #PWR0103
+U 1 1 5E66ACD7
+P 8050 4300
+F 0 "#PWR0103" H 8050 4150 50  0001 C CNN
+F 1 "-BATT" H 8065 4473 50  0000 C CNN
+F 2 "" H 8050 4300 50  0001 C CNN
+F 3 "" H 8050 4300 50  0001 C CNN
+	1    8050 4300
+	-1   0    0    1
+$EndComp
+$Comp
+L power:GND #PWR0104
+U 1 1 5E670334
+P 5950 4300
+F 0 "#PWR0104" H 5950 4050 50  0001 C CNN
+F 1 "GND" H 5955 4127 50  0000 C CNN
+F 2 "" H 5950 4300 50  0001 C CNN
+F 3 "" H 5950 4300 50  0001 C CNN
+	1    5950 4300
+	1    0    0    -1
+$EndComp
+Wire Wire Line
+	5950 3950 5950 4300
+$Comp
+L power:-BATT #PWR0105
+U 1 1 5E6750F4
+P 6450 4000
+F 0 "#PWR0105" H 6450 3850 50  0001 C CNN
+F 1 "-BATT" H 6465 4173 50  0000 C CNN
+F 2 "" H 6450 4000 50  0001 C CNN
+F 3 "" H 6450 4000 50  0001 C CNN
+	1    6450 4000
+	-1   0    0    1
+$EndComp
+$Comp
+L power:-BATT #PWR0106
+U 1 1 5E675645
+P 5500 3800
+F 0 "#PWR0106" H 5500 3650 50  0001 C CNN
+F 1 "-BATT" H 5515 3973 50  0000 C CNN
+F 2 "" H 5500 3800 50  0001 C CNN
+F 3 "" H 5500 3800 50  0001 C CNN
+	1    5500 3800
+	-1   0    0    1
+$EndComp
+$Comp
+L power:GND #PWR0107
+U 1 1 5E676144
+P 3500 4950
+F 0 "#PWR0107" H 3500 4700 50  0001 C CNN
+F 1 "GND" H 3505 4777 50  0000 C CNN
+F 2 "" H 3500 4950 50  0001 C CNN
+F 3 "" H 3500 4950 50  0001 C CNN
+	1    3500 4950
+	1    0    0    -1
+$EndComp
+$Comp
+L power:GND #PWR0108
+U 1 1 5E676C0E
+P 2650 4850
+F 0 "#PWR0108" H 2650 4600 50  0001 C CNN
+F 1 "GND" H 2655 4677 50  0000 C CNN
+F 2 "" H 2650 4850 50  0001 C CNN
+F 3 "" H 2650 4850 50  0001 C CNN
+	1    2650 4850
+	1    0    0    -1
+$EndComp
+$Comp
+L power:GND #PWR0109
+U 1 1 5E67AF77
+P 2000 5000
+F 0 "#PWR0109" H 2000 4750 50  0001 C CNN
+F 1 "GND" H 2005 4827 50  0000 C CNN
+F 2 "" H 2000 5000 50  0001 C CNN
+F 3 "" H 2000 5000 50  0001 C CNN
+	1    2000 5000
+	1    0    0    -1
+$EndComp
+$Comp
+L power:GND #PWR0110
+U 1 1 5E67F28A
+P 1600 5000
+F 0 "#PWR0110" H 1600 4750 50  0001 C CNN
+F 1 "GND" H 1605 4827 50  0000 C CNN
+F 2 "" H 1600 5000 50  0001 C CNN
+F 3 "" H 1600 5000 50  0001 C CNN
+	1    1600 5000
+	1    0    0    -1
+$EndComp
+$Comp
+L power:GND #PWR0111
+U 1 1 5E683611
+P 3850 4250
+F 0 "#PWR0111" H 3850 4000 50  0001 C CNN
+F 1 "GND" H 3855 4077 50  0000 C CNN
+F 2 "" H 3850 4250 50  0001 C CNN
+F 3 "" H 3850 4250 50  0001 C CNN
+	1    3850 4250
+	1    0    0    -1
+$EndComp
+$Comp
+L power:GND #PWR0112
+U 1 1 5E687951
+P 3600 3750
+F 0 "#PWR0112" H 3600 3500 50  0001 C CNN
+F 1 "GND" H 3605 3577 50  0000 C CNN
+F 2 "" H 3600 3750 50  0001 C CNN
+F 3 "" H 3600 3750 50  0001 C CNN
+	1    3600 3750
+	1    0    0    -1
+$EndComp
+$Comp
+L power:GND #PWR0113
+U 1 1 5E68BE40
+P 1400 4300
+F 0 "#PWR0113" H 1400 4050 50  0001 C CNN
+F 1 "GND" H 1405 4127 50  0000 C CNN
+F 2 "" H 1400 4300 50  0001 C CNN
+F 3 "" H 1400 4300 50  0001 C CNN
+	1    1400 4300
+	1    0    0    -1
+$EndComp
+$Comp
+L power:GND #PWR0114
+U 1 1 5E690329
+P 1200 1700
+F 0 "#PWR0114" H 1200 1450 50  0001 C CNN
+F 1 "GND" H 1205 1527 50  0000 C CNN
+F 2 "" H 1200 1700 50  0001 C CNN
+F 3 "" H 1200 1700 50  0001 C CNN
+	1    1200 1700
+	1    0    0    -1
+$EndComp
+$Comp
+L power:GND #PWR0115
+U 1 1 5E6947C8
+P 2000 1450
+F 0 "#PWR0115" H 2000 1200 50  0001 C CNN
+F 1 "GND" H 2005 1277 50  0000 C CNN
+F 2 "" H 2000 1450 50  0001 C CNN
+F 3 "" H 2000 1450 50  0001 C CNN
+	1    2000 1450
+	1    0    0    -1
+$EndComp
 $EndSCHEMATC
