File: Hardware/MainPCB/MainPCB.sch (KiCad schematic (older format))
At the start: 31 parts, among them J1 USB_B_Micro, Q1 NTR2101P, Q2 FDS9926A, U1 BQ24075, U2 BQ29700, U3 TLV75533PDBV

Commit message: Finished MainPCB + generated gerber files + aanpassingen BOM
Connections:
- net GND: now also C3.2
Changed lines of the file:
@@
+	1    0    0    -1
+$EndComp
+$Comp
+L power:GND #PWR?
+U 1 1 5E702652
+P 2400 3300
+F 0 "#PWR?" H 2400 3050 50  0001 C CNN
+F 1 "GND" H 2405 3127 50  0000 C CNN
+F 2 "" H 2400 3300 50  0001 C CNN
+F 3 "" H 2400 3300 50  0001 C CNN
+	1    2400 3300
 	1    0    0    -1
 $EndComp

Commit message: BOM list mainPCB
Parts:
- D1: value LED_Green -> TLHG44K1L2
- D2: value LED_Blue -> TLHB44K2M1
Changed lines of the file:
@@
 P 4300 4250
 F 0 "D1" V 4339 4133 50  0000 R CNN
-F 1 "LED_Green" V 4248 4133 50  0000 R CNN
+F 1 "TLHG44K1L2" V 4248 4133 50  0000 R CNN
 F 2 "LED_THT:LED_D3.0mm" H 4300 4250 50  0001 C CNN
 F 3 "~" H 4300 4250 50  0001 C CNN
@@
 P 4650 4250
 F 0 "D2" V 4689 4133 50  0000 R CNN
-F 1 "LED_Blue" V 4598 4133 50  0000 R CNN
+F 1 "TLHB44K2M1" V 4598 4133 50  0000 R CNN
 F 2 "LED_THT:LED_D3.0mm" H 4650 4250 50  0001 C CNN
 F 3 "~" H 4650 4250 50  0001 C CNN
@@
 $EndComp
 $Comp
-L power:GND #PWR?
+L power:GND #PWR0116
 U 1 1 5E702652
 P 2400 3300
-F 0 "#PWR?" H 2400 3050 50  0001 C CNN
+F 0 "#PWR0116" H 2400 3050 50  0001 C CNN
 F 1 "GND" H 2405 3127 50  0000 C CNN
 F 2 "" H 2400 3300 50  0001 C CNN
