File: Hardware/SensorBoard/SesnorBoard/SesnorBoard.sch (KiCad schematic (older format))
At the start: 31 parts, among them J1 Mainboard connection, J2 microphoon connection, U1 AMG8833, U2 CCS811, U3 NC7SVU04P5X

Commit message: Eerste pcb layouts ensorboard
Parts:
- removed R3, R4: 2k2, Resistor_SMD:R_1206_3216Metric, symbol SesnorBoard-eagle-import:RESISTOR_1206
- C1, C11, C2, C21, C3, C6: footprint Capacitor_SMD:C_1206_3216Metric -> Capacitor_SMD:C_0805_2012Metric; symbol SesnorBoard-eagle-import:CAP_CERAMIC_1206 -> SesnorBoard-eagle-import:CAP_CERAMIC0805-NOOUTLINE
- J1: footprint Connector_PinHeader_1.00mm:PinHeader_1x08_P1.00mm_Vertical -> Connector_PinHeader_1.00mm:PinHeader_1x09_P1.00mm_Vertical; symbol Connector_Generic:Conn_01x08 -> Connector_Generic:Conn_01x09
- R1, R11, R12, R13, R14, R15, R16, R2, R21, R5: footprint Resistor_SMD:R_1206_3216Metric -> Resistor_SMD:R_0805_2012Metric; symbol SesnorBoard-eagle-import:RESISTOR_1206 -> SesnorBoard-eagle-import:RESISTOR0805_NOOUTLINE
- TH1: footprint Resistor_SMD:R_0603_1608Metric -> (none)
- U1: footprint AMG8833_REV-B:AMG8833 -> SesnorBoard:AMG8833
Connections:
- net labels added: +3.3V, AUX, DETECTOR-OUT, INT_CSS811
- wire segments 95 -> 91
Other:
- note added: "C11 zo kort mogelijk \nbij voedingspin VDD (6)"
- note removed: "Place C11 as close as possible \nto the supply pin VDD (6)"
