File: Hardware/SesnorBoard/_autosave-SesnorBoard.sch (KiCad schematic (older format))
At the start: 29 parts, among them J1 Mainboard connection, J2 microphoon connection, U1 AMG8833, U2 CCS811, U3 NC7SVU04P5X

Commit message: Eerste pcb layouts ensorboard
Parts:
- added R3, R4: 2k2, Resistor_SMD:R_1206_3216Metric, symbol SesnorBoard-eagle-import:RESISTOR_1206
- C1, C11, C2, C21, C3, C6: footprint Capacitor_SMD:C_0805_2012Metric -> Capacitor_SMD:C_1206_3216Metric; symbol SesnorBoard-eagle-import:CAP_CERAMIC0805-NOOUTLINE -> SesnorBoard-eagle-import:CAP_CERAMIC_1206
- D1: symbol SesnorBoard-rescue:PMEG4050EP-Diode -> Diode:PMEG4050EP
- J1: footprint Connector_PinHeader_1.00mm:PinHeader_1x09_P1.00mm_Vertical -> Connector_PinHeader_1.00mm:PinHeader_1x08_P1.00mm_Vertical; symbol Connector_Generic:Conn_01x09 -> Connector_Generic:Conn_01x08
- R1, R11, R12, R13, R14, R15, R16, R2, R21, R5: footprint Resistor_SMD:R_0805_2012Metric -> Resistor_SMD:R_1206_3216Metric; symbol SesnorBoard-eagle-import:RESISTOR0805_NOOUTLINE -> SesnorBoard-eagle-import:RESISTOR_1206
- TH1: footprint (none) -> Resistor_SMD:R_1206_3216Metric
- U1: footprint SesnorBoard:AMG8833 -> AMG8833_REV-B:AMG8833
Connections:
- net labels removed: +3.3V, AUX, DETECTOR-OUT, INT_CSS811
- wire segments 91 -> 95
