File: Hardware/SesnorBoard/SesnorBoard.kicad_pcb (KiCad board)
At the start: 2 copper layers, 39.4 x 31.1 mm, 25 parts, among them J1 Mainboard connection, J2 microphoon connection, U1 AMG8833, U2 CCS811, U3 NC7SVU04P5X

Commit message: updated the sensor part of the report and corrected some issues of the PCB design.
Parts:
- J2: footprint Connector_PinHeader_2.00mm:PinHeader_1x03_P2.00mm_Vertical -> Connector_PinHeader_2.54mm:PinHeader_1x03_P2.54mm_Vertical
- R21: value 100k -> 1M
- moved C21 0.64 mm to (50.8, -297.8)
- moved R21 0.64 mm to (50.8, -295.3)
- moved D1 0.63 mm to (49.8, -292.7)
- moved J2 0.63 mm to (47.5, -287.7)
Routing:
- net /AUDIO_3V3: track 8.58 -> 17.8 mm
- net GND: track 100.4 -> 96.9 mm
- removed copper zone on B.Cu, net /AUDIO_3V3
